File: hardware/pcb and schematic desing/pcb milton/fotosintX/fotosintX.kicad_pcb (KiCad board)
At the start: 2 copper layers, 46.5 x 74.3 mm, 12 parts, among them J4 TB_1X2, J5 TB_1X2, Q1 2N3904, U1 ESP32_DEVKITC, U2 L7805

Commit message: Mejorando pcb
Parts:
- added D1: 1N4007, Diode_THT:D_DO-41_SOD81_P10.16mm_Horizontal, F.Cu at (193.1, 101.4)
- added H1: Mounting_Hole, eestn5:hole_3mm, F.Cu at (202.9, 113.4)
- added H2: Mounting_Hole, eestn5:hole_3mm, F.Cu at (172.1, 47.3)
- C1, C2: footprint eestn5:CAP_ELEC_8x11.5mm -> eestn5:CAP_0.1
- Q1: value 2N3904 -> PN2222A; footprint Package_TO_SOT_THT:TO-92_Inline -> Package_TO_SOT_THT:TO-92_Wide
- moved Q1 21.3 mm to (191.1, 85.7), turned to 180 degrees
- moved C1 8.95 mm to (172.4, 115.0), turned to 0 degrees
- moved LCDOLED1 8.26 mm to (191.3, 45.8), turned to 180 degrees
- moved C2 7.07 mm to (172.3, 101.6), turned to 180 degrees
- moved LDRMODULO1 4.88 mm to (191.2, 50.8), turned to 180 degrees
- moved R1 4.21 mm to (192.4, 91.5), turned to 0 degrees
- moved J4 2.93 mm to (193.9, 108.9)
- moved SENSORNIVELDEAGUA1 2.38 mm to (184.4, 48.2)
- moved SENSORHUMEDAD1 0.95 mm to (181.0, 48.2)
- moved J5 0.34 mm to (180.4, 108.9)
- moved U2 0.21 mm to (172.4, 108.3)
Connections:
- J4 pad 1: /motor -> +5V
- LCDOLED1 pad 1: /SDA -> /SCL
- LCDOLED1 pad 2: /SCL -> /SDA
- Q1 pad 3: /motor -> +5V
Routing:
- net Net-(Q1-B): track 11.5 -> 3.27 mm
- net +5V: track 101.9 -> 109.7 mm
- net /motor: track 5.50 -> 0.00 mm
- net /SDA: track 33.9 -> 37.9 mm
- net /ON: track 5.08 -> 3.20 mm
- net /SERIAL: track 24.9 -> 23.3 mm
- net +12V: track 12.2 -> 11.0 mm
- net /AUOT: track 18.7 -> 18.0 mm
- net /SCL: track 20.8 -> 21.4 mm
Other:
- board size 46.5 x 74.3 mm -> 39 x 76 mm

Commit message: pcb modified
Parts:
- added J1: Conn_01x02_Pin, Connector_PinHeader_2.54mm:PinHeader_1x02_P2.54mm_Vertical, F.Cu at (203.2, 108.0)
- R1: value R -> 1500
- renumbered SENSORNIVELDEAGUA1 to CAUDALIMETRO1
Connections:
- D1 pad 2: +5V -> /motor-
- Q1 pad 3: +5V -> /motor-
Routing:
- net /motor-: track 0.00 -> 44.8 mm
- net +5V: track 109.7 -> 116.1 mm
- net /SDA: track 37.9 -> 38.7 mm

Commit message: add pcb printing pdf
Parts:
- H2: moved to B.Cu
- turned H2 to 180 degrees
Changed lines of the file:
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@@
-    )
-  )
-  (footprint "eestn5:hole_3mm" (layer "F.Cu")
-    (at 172.1 47.3)
-    (descr "Hole 3mm")
-    (property "Sheetfile" "fotosintX.kicad_sch")
-    (property "Sheetname" "")
-    (property "ki_description" "Mounting Hole without connection")
-    (property "ki_keywords" "mounting hole")
-    (attr through_hole)
-    (fp_text reference "H2" (at 0 -3.302) (layer "F.SilkS") hide
-        (effects (font (size 1.524 1.524) (thickness 0.3048)))
-    )
-    (fp_text value "Mounting_Hole" (at 5.334 0) (layer "F.SilkS") hide
-        (effects (font (size 1.524 1.524) (thickness 0.3048)))
-    )
-    (fp_line (start -3 0) (end 3 0)
-      (stroke (width 0.254) (type solid)) (layer "B.SilkS"))
-    (fp_line (start 0 -3) (end 0 3)
-      (stroke (width 0.254) (type solid)) (layer "B.SilkS"))
-    (fp_circle (center 0 0) (end 3 0)
-      (stroke (width 0.254) (type solid)) (fill none) (layer "B.SilkS"))
-    (fp_line (start -3 0) (end 3 0)
-      (stroke (width 0.254) (type solid)) (layer "F.SilkS"))
-    (fp_line (start 0 -3) (end 0 3)
-      (stroke (width 0.254) (type solid)) (layer "F.SilkS"))
-    (fp_circle (center 0 0) (end 3 0)
-      (stroke (width 0.254) (type solid)) (fill none) (layer "F.SilkS"))
-    (pad "" np_thru_hole circle (at 0 0) (size 3 3) (drill 3) (layers "F&B.Cu" "*.Mask"))
-    (model "C:/EESTN5/Librerias-Kicad-master/EESTN5.3dshapes/Tornillo_M3_8mm_Tuerca.wrl"
-      (offset (xyz 0 0 0))
-      (scale (xyz 1 1 1))
-      (rotate (xyz 0 0 0))
     )
   )
@@
       (scale (xyz 0.3937 0.3937 0.3937))
       (rotate (xyz 0 -90 180))
+    )
+  )
+  (footprint "eestn5:hole_3mm" (layer "B.Cu")
+    (at 172.1 47.3 180)
+    (descr "Hole 3mm")
+    (property "Sheetfile" "fotosintX.kicad_sch")
+    (property "Sheetname" "")
+    (property "ki_description" "Mounting Hole without connection")
+    (property "ki_keywords" "mounting hole")
+    (attr through_hole)
+    (fp_text reference "H2" (at 0 3.302) (layer "B.SilkS") hide
+        (effects (font (size 1.524 1.524) (thickness 0.3048)) (justify mirror))
+    )
+    (fp_text value "Mounting_Hole" (at 5.334 0) (layer "B.SilkS") hide
+        (effects (font (size 1.524 1.524) (thickness 0.3048)) (justify mirror))
+    )
+    (fp_line (start -3 0) (end 3 0)
+      (stroke (width 0.254) (type solid)) (layer "B.SilkS"))
+    (fp_line (start 0 3) (end 0 -3)
+      (stroke (width 0.254) (type solid)) (layer "B.SilkS"))
+    (fp_circle (center 0 0) (end 3 0)
+      (stroke (width 0.254) (type solid)) (fill none) (layer "B.SilkS"))
+    (fp_line (start -3 0) (end 3 0)
+      (stroke (width 0.254) (type solid)) (layer "F.SilkS"))
+    (fp_line (start 0 3) (end 0 -3)
+      (stroke (width 0.254) (type solid)) (layer "F.SilkS"))
+    (fp_circle (center 0 0) (end 3 0)
+      (stroke (width 0.254) (type solid)) (fill none) (layer "F.SilkS"))
+    (pad "" np_thru_hole circle (at 0 0 180) (size 3 3) (drill 3) (layers "F&B.Cu" "*.Mask"))
+    (model "C:/EESTN5/Librerias-Kicad-master/EESTN5.3dshapes/Tornillo_M3_8mm_Tuerca.wrl"
+      (offset (xyz 0 0 0))
+      (scale (xyz 1 1 1))
+      (rotate (xyz 0 0 0))
     )
   )
@@
     (connect_pads (clearance 0.5))
     (min_thickness 0.3) (filled_areas_thickness no)
-    (fill yes (thermal_gap 0.5) (thermal_bridge_width 0.5))
+    (fill yes (thermal_gap 0.5) (thermal_bridge_width 0.8))
     (polygon
       (pts

Commit message: PCB terminado
Parts:
- removed J5: TB_1X2, eestn5:BORNERA2
- added C1: 0,33uF, eestn5:CAP_0.1, F.Cu at (231.6, 186.3)
- added C1: 0,33uF, eestn5:CAP_0.1, F.Cu at (229.9, 93.1)
- added C1: 0,33uF, eestn5:CAP_0.1, F.Cu at (127.9, 187.4)
- added C1: 0,33uF, eestn5:CAP_0.1, F.Cu at (177.0, 94.2)
- added C1: 0,33uF, eestn5:CAP_0.1, F.Cu at (124.3, 93.9)
- added C1: 0,33uF, eestn5:CAP_0.1, F.Cu at (22.3, 94.0)
- added C1: 0,33uF, eestn5:CAP_0.1, F.Cu at (75.2, 187.1)
- added C1: 0,33uF, eestn5:CAP_0.1, F.Cu at (75.0, 94.3)
- added C1: 0,33uF, eestn5:CAP_0.1, F.Cu at (178.9, 186.0)
- added C2: 0,1uF, eestn5:CAP_0.1, F.Cu at (178.8, 172.6)
- added C2: 0,1uF, eestn5:CAP_0.1, F.Cu at (229.8, 79.7)
- added C2: 0,1uF, eestn5:CAP_0.1, F.Cu at (75.1, 173.7)
- added C2: 0,1uF, eestn5:CAP_0.1, F.Cu at (127.8, 174.0)
- added C2: 0,1uF, eestn5:CAP_0.1, F.Cu at (176.9, 80.8)
- added C2: 0,1uF, eestn5:CAP_0.1, F.Cu at (231.5, 172.9)
- added C2: 0,1uF, eestn5:CAP_0.1, F.Cu at (124.2, 80.5)
- added C2: 0,1uF, eestn5:CAP_0.1, F.Cu at (22.2, 80.6)
- added C2: 0,1uF, eestn5:CAP_0.1, F.Cu at (74.9, 80.9)
- added CAUDALIMETRO1: Conn_01X03, eestn5:Pin_Strip_3, F.Cu at (136.3, 27.1)
- added CAUDALIMETRO1: Conn_01X03, eestn5:Pin_Strip_3, F.Cu at (139.9, 120.6)
- added CAUDALIMETRO1: Conn_01X03, eestn5:Pin_Strip_3, F.Cu at (243.6, 119.5)
- added CAUDALIMETRO1: Conn_01X03, eestn5:Pin_Strip_3, F.Cu at (189.0, 27.4)
- added CAUDALIMETRO1: Conn_01X03, eestn5:Pin_Strip_3, F.Cu at (87.0, 27.5)
- added CAUDALIMETRO1: Conn_01X03, eestn5:Pin_Strip_3, F.Cu at (190.9, 119.2)
- added CAUDALIMETRO1: Conn_01X03, eestn5:Pin_Strip_3, F.Cu at (241.9, 26.3)
- added CAUDALIMETRO1: Conn_01X03, eestn5:Pin_Strip_3, F.Cu at (87.2, 120.3)
- added CAUDALIMETRO1: Conn_01X03, eestn5:Pin_Strip_3, F.Cu at (34.3, 27.2)
- added D1: 1N4007, Diode_THT:D_DO-41_SOD81_P10.16mm_Horizontal, F.Cu at (199.6, 172.4)
- added D1: 1N4007, Diode_THT:D_DO-41_SOD81_P10.16mm_Horizontal, F.Cu at (252.3, 172.7)
- added D1: 1N4007, Diode_THT:D_DO-41_SOD81_P10.16mm_Horizontal, F.Cu at (197.7, 80.6)
- added D1: 1N4007, Diode_THT:D_DO-41_SOD81_P10.16mm_Horizontal, F.Cu at (148.6, 173.8)
- added D1: 1N4007, Diode_THT:D_DO-41_SOD81_P10.16mm_Horizontal, F.Cu at (145.0, 80.3)
- added D1: 1N4007, Diode_THT:D_DO-41_SOD81_P10.16mm_Horizontal, F.Cu at (95.7, 80.7)
- added D1: 1N4007, Diode_THT:D_DO-41_SOD81_P10.16mm_Horizontal, F.Cu at (43.0, 80.4)
- added D1: 1N4007, Diode_THT:D_DO-41_SOD81_P10.16mm_Horizontal, F.Cu at (250.6, 79.5)
- added D1: 1N4007, Diode_THT:D_DO-41_SOD81_P10.16mm_Horizontal, F.Cu at (95.9, 173.5)
- added H1: Mounting_Hole, eestn5:hole_3mm, F.Cu at (209.4, 184.4)
- added H1: Mounting_Hole, eestn5:hole_3mm, F.Cu at (105.5, 92.7)
- added H1: Mounting_Hole, eestn5:hole_3mm, F.Cu at (262.1, 184.7)
- added H1: Mounting_Hole, eestn5:hole_3mm, F.Cu at (158.4, 185.8)
- added H1: Mounting_Hole, eestn5:hole_3mm, F.Cu at (207.5, 92.6)
- added H1: Mounting_Hole, eestn5:hole_3mm, F.Cu at (105.7, 185.5)
- added H1: Mounting_Hole, eestn5:hole_3mm, F.Cu at (52.8, 92.4)
- added H1: Mounting_Hole, eestn5:hole_3mm, F.Cu at (260.4, 91.5)
- added H1: Mounting_Hole, eestn5:hole_3mm, F.Cu at (154.8, 92.3)
- added H2: Mounting_Hole, eestn5:hole_3mm, B.Cu at (74.9, 119.4)
- added H2: Mounting_Hole, eestn5:hole_3mm, B.Cu at (231.3, 118.6)
- added H2: Mounting_Hole, eestn5:hole_3mm, B.Cu at (74.7, 26.6)
- added H2: Mounting_Hole, eestn5:hole_3mm, B.Cu at (229.6, 25.4)
- added H2: Mounting_Hole, eestn5:hole_3mm, B.Cu at (178.6, 118.3)
- added H2: Mounting_Hole, eestn5:hole_3mm, B.Cu at (22.0, 26.3)
- added H2: Mounting_Hole, eestn5:hole_3mm, B.Cu at (127.6, 119.7)
- added H2: Mounting_Hole, eestn5:hole_3mm, B.Cu at (124.0, 26.2)
- added H2: Mounting_Hole, eestn5:hole_3mm, B.Cu at (176.7, 26.5)
- added J1: Conn_01x02_Pin, Connector_PinHeader_2.54mm:PinHeader_1x02_P2.54mm_Vertical, F.Cu at (158.7, 180.3)
- added J1: Conn_01x02_Pin, Connector_PinHeader_2.54mm:PinHeader_1x02_P2.54mm_Vertical, F.Cu at (207.8, 87.2)
- added J1: Conn_01x02_Pin, Connector_PinHeader_2.54mm:PinHeader_1x02_P2.54mm_Vertical, F.Cu at (260.7, 86.0)
- added J1: Conn_01x02_Pin, Connector_PinHeader_2.54mm:PinHeader_1x02_P2.54mm_Vertical, F.Cu at (209.7, 178.9)
- added J1: Conn_01x02_Pin, Connector_PinHeader_2.54mm:PinHeader_1x02_P2.54mm_Vertical, F.Cu at (106.0, 180.1)
- added J1: Conn_01x02_Pin, Connector_PinHeader_2.54mm:PinHeader_1x02_P2.54mm_Vertical, F.Cu at (155.1, 86.8)
- added J1: Conn_01x02_Pin, Connector_PinHeader_2.54mm:PinHeader_1x02_P2.54mm_Vertical, F.Cu at (53.1, 87.0)
- added J1: Conn_01x02_Pin, Connector_PinHeader_2.54mm:PinHeader_1x02_P2.54mm_Vertical, F.Cu at (105.8, 87.2)
- added J1: Conn_01x02_Pin, Connector_PinHeader_2.54mm:PinHeader_1x02_P2.54mm_Vertical, F.Cu at (262.4, 179.2)
- added J2: Jack-DC, jack dc 12v 2 patas:CUI_PJ-037AH, F.Cu at (30.8, 179.4)
- added J2: Jack-DC, jack dc 12v 2 patas:CUI_PJ-037AH, F.Cu at (136.6, 179.9)
- added J2: Jack-DC, jack dc 12v 2 patas:CUI_PJ-037AH, F.Cu at (133.0, 86.4)
- added J2: Jack-DC, jack dc 12v 2 patas:CUI_PJ-037AH, F.Cu at (240.3, 178.8)
- added J2: Jack-DC, jack dc 12v 2 patas:CUI_PJ-037AH, F.Cu at (83.9, 179.6)
- added J2: Jack-DC, jack dc 12v 2 patas:CUI_PJ-037AH, F.Cu at (238.6, 85.6)
- added J2: Jack-DC, jack dc 12v 2 patas:CUI_PJ-037AH, F.Cu at (185.7, 86.7)
- added J2: Jack-DC, jack dc 12v 2 patas:CUI_PJ-037AH, F.Cu at (187.6, 178.5)
- added J2: Jack-DC, jack dc 12v 2 patas:CUI_PJ-037AH, F.Cu at (31.0, 86.5)
- added J2: Jack-DC, jack dc 12v 2 patas:CUI_PJ-037AH, F.Cu at (83.7, 86.8)
- added J4: TB_1X2, eestn5:BORNERA2, F.Cu at (199.7, 183.2)
- added J4: TB_1X2, eestn5:BORNERA2, F.Cu at (43.1, 91.2)
- added J4: TB_1X2, eestn5:BORNERA2, F.Cu at (148.7, 184.6)
- added J4: TB_1X2, eestn5:BORNERA2, F.Cu at (252.4, 183.5)
- added J4: TB_1X2, eestn5:BORNERA2, F.Cu at (95.8, 91.5)
- added J4: TB_1X2, eestn5:BORNERA2, F.Cu at (197.8, 91.4)
- added J4: TB_1X2, eestn5:BORNERA2, F.Cu at (250.7, 90.3)
- added J4: TB_1X2, eestn5:BORNERA2, F.Cu at (145.1, 91.1)
- added J4: TB_1X2, eestn5:BORNERA2, F.Cu at (96.0, 184.3)
- added LCDOLED1: Conn_01x04, eestn5:pin_strip_4, F.Cu at (94.1, 117.9)
- added LCDOLED1: Conn_01x04, eestn5:pin_strip_4, F.Cu at (250.5, 117.1)
- added LCDOLED1: Conn_01x04, eestn5:pin_strip_4, F.Cu at (143.2, 24.7)
- added LCDOLED1: Conn_01x04, eestn5:pin_strip_4, F.Cu at (248.8, 23.9)
- added LCDOLED1: Conn_01x04, eestn5:pin_strip_4, F.Cu at (41.2, 24.8)
- added LCDOLED1: Conn_01x04, eestn5:pin_strip_4, F.Cu at (197.8, 116.8)
- added LCDOLED1: Conn_01x04, eestn5:pin_strip_4, F.Cu at (93.9, 25.1)
- added LCDOLED1: Conn_01x04, eestn5:pin_strip_4, F.Cu at (195.9, 25.0)
- added LCDOLED1: Conn_01x04, eestn5:pin_strip_4, F.Cu at (146.8, 118.2)
- added LDRMODULO1: Conn_01x04, eestn5:pin_strip_4, F.Cu at (195.8, 30.0)
- added LDRMODULO1: Conn_01x04, eestn5:pin_strip_4, F.Cu at (248.7, 28.9)
- added LDRMODULO1: Conn_01x04, eestn5:pin_strip_4, F.Cu at (197.7, 121.8)
- added LDRMODULO1: Conn_01x04, eestn5:pin_strip_4, F.Cu at (93.8, 30.1)
- added LDRMODULO1: Conn_01x04, eestn5:pin_strip_4, F.Cu at (143.1, 29.7)
- added LDRMODULO1: Conn_01x04, eestn5:pin_strip_4, F.Cu at (94.0, 122.9)
- added LDRMODULO1: Conn_01x04, eestn5:pin_strip_4, F.Cu at (146.7, 123.2)
- added LDRMODULO1: Conn_01x04, eestn5:pin_strip_4, F.Cu at (250.4, 122.1)
- added LDRMODULO1: Conn_01x04, eestn5:pin_strip_4, F.Cu at (41.1, 29.8)
- added Q1: PN2222A, Package_TO_SOT_THT:TO-92_Wide, F.Cu at (248.6, 63.8)
- added Q1: PN2222A, Package_TO_SOT_THT:TO-92_Wide, F.Cu at (146.6, 158.1)
- added Q1: PN2222A, Package_TO_SOT_THT:TO-92_Wide, F.Cu at (41.0, 64.7)
- added Q1: PN2222A, Package_TO_SOT_THT:TO-92_Wide, F.Cu at (93.7, 65.0)
- added Q1: PN2222A, Package_TO_SOT_THT:TO-92_Wide, F.Cu at (143.0, 64.6)
- added Q1: PN2222A, Package_TO_SOT_THT:TO-92_Wide, F.Cu at (197.6, 156.7)
- added Q1: PN2222A, Package_TO_SOT_THT:TO-92_Wide, F.Cu at (93.9, 157.8)
- added Q1: PN2222A, Package_TO_SOT_THT:TO-92_Wide, F.Cu at (195.7, 64.9)
- added Q1: PN2222A, Package_TO_SOT_THT:TO-92_Wide, F.Cu at (250.3, 157.0)
- added R1: 1500, eestn5:RES0.3, F.Cu at (144.3, 70.4)
- added R1: 1500, eestn5:RES0.3, F.Cu at (249.9, 69.6)
- added R1: 1500, eestn5:RES0.3, F.Cu at (147.9, 163.9)
- added R1: 1500, eestn5:RES0.3, F.Cu at (42.3, 70.5)
- added R1: 1500, eestn5:RES0.3, F.Cu at (251.6, 162.8)
- added R1: 1500, eestn5:RES0.3, F.Cu at (197.0, 70.7)
- added R1: 1500, eestn5:RES0.3, F.Cu at (95.2, 163.6)
- added R1: 1500, eestn5:RES0.3, F.Cu at (95.0, 70.8)
- added R1: 1500, eestn5:RES0.3, F.Cu at (198.9, 162.5)
- added SENSORHUMEDAD1: Conn_01X03, eestn5:Pin_Strip_3, F.Cu at (136.5, 120.6)
- added SENSORHUMEDAD1: Conn_01X03, eestn5:Pin_Strip_3, F.Cu at (240.2, 119.5)
- added SENSORHUMEDAD1: Conn_01X03, eestn5:Pin_Strip_3, F.Cu at (187.5, 119.2)
- added SENSORHUMEDAD1: Conn_01X03, eestn5:Pin_Strip_3, F.Cu at (83.8, 120.3)
- added SENSORHUMEDAD1: Conn_01X03, eestn5:Pin_Strip_3, F.Cu at (132.9, 27.1)
- added SENSORHUMEDAD1: Conn_01X03, eestn5:Pin_Strip_3, F.Cu at (185.6, 27.4)
- added SENSORHUMEDAD1: Conn_01X03, eestn5:Pin_Strip_3, F.Cu at (83.6, 27.5)
- added SENSORHUMEDAD1: Conn_01X03, eestn5:Pin_Strip_3, F.Cu at (30.9, 27.2)
- added SENSORHUMEDAD1: Conn_01X03, eestn5:Pin_Strip_3, F.Cu at (238.5, 26.3)
- added U1: ESP32_DEVKITC, eestn5:ESP32S, F.Cu at (37.9, 57.7)
- added U1: ESP32_DEVKITC, eestn5:ESP32S, F.Cu at (90.6, 58.0)
- added U1: ESP32_DEVKITC, eestn5:ESP32S, F.Cu at (194.5, 149.7)
- added U1: ESP32_DEVKITC, eestn5:ESP32S, F.Cu at (192.6, 57.9)
- added U1: ESP32_DEVKITC, eestn5:ESP32S, F.Cu at (90.8, 150.8)
- added U1: ESP32_DEVKITC, eestn5:ESP32S, F.Cu at (245.5, 56.8)
- added U1: ESP32_DEVKITC, eestn5:ESP32S, F.Cu at (139.9, 57.6)
- added U1: ESP32_DEVKITC, eestn5:ESP32S, F.Cu at (143.5, 151.1)
- added U1: ESP32_DEVKITC, eestn5:ESP32S, F.Cu at (247.2, 150.0)
- added U2: L7805, eestn5:TO-220, F.Cu at (22.3, 87.3)
- added U2: L7805, eestn5:TO-220, F.Cu at (229.9, 86.4)
- added U2: L7805, eestn5:TO-220, F.Cu at (75.0, 87.6)
- added U2: L7805, eestn5:TO-220, F.Cu at (178.9, 179.3)
- added U2: L7805, eestn5:TO-220, F.Cu at (75.2, 180.4)
- added U2: L7805, eestn5:TO-220, F.Cu at (177.0, 87.5)
- added U2: L7805, eestn5:TO-220, F.Cu at (127.9, 180.7)
- added U2: L7805, eestn5:TO-220, F.Cu at (231.6, 179.6)
- added U2: L7805, eestn5:TO-220, F.Cu at (124.3, 87.2)
- moved J4 168.7 mm to (42.9, 184.1)
- moved C1 166.6 mm to (22.1, 186.9)
- moved C2 166.6 mm to (22.0, 173.5)
- moved D1 166.6 mm to (42.8, 173.3)
- moved H1 166.6 mm to (52.6, 185.3)
- moved LCDOLED1 166.6 mm to (41.0, 117.7)
- moved LDRMODULO1 166.6 mm to (40.9, 122.7)
- moved Q1 166.6 mm to (40.8, 157.6)
- moved R1 166.6 mm to (42.1, 163.4)
- moved SENSORHUMEDAD1 166.6 mm to (30.7, 120.1)
- moved U1 166.6 mm to (37.7, 150.6)
- moved U2 166.6 mm to (22.1, 180.2)
- moved CAUDALIMETRO1 166.6 mm to (34.1, 120.1)
- moved H2 166.6 mm to (21.8, 119.2)
- moved J1 166.6 mm to (52.9, 179.8)
Connections:
- LCDOLED1 pad 1: /SCL -> /SDA
- LCDOLED1 pad 2: /SDA -> /SCL
- LDRMODULO1 pad 4: +5V -> +3.3V
- U1 pad 1: unconnected-(U1-3V3-Pad1) -> +3.3V
- U1 pad 5: /AUOT -> /SERIAL
- U1 pad 6: /SERIAL -> /AUOT
Routing:
- net +5V: track 116.1 -> 1406.2 mm
- net /motor-: track 44.8 -> 450.9 mm
- net /A0: track 33.0 -> 329.9 mm
- net /SDA: track 38.7 -> 325.2 mm
- net /AUOT: track 18.0 -> 289.6 mm
- net /SERIAL: track 23.3 -> 267.6 mm
- net /SCL: track 21.4 -> 238.1 mm
- net +3.3V: track 0.00 -> 145.2 mm
- net +12V: track 11.0 -> 147.9 mm
- net Net-(Q1-B): track 3.27 -> 32.7 mm
- net /ON: track 3.20 -> 32.0 mm
Other:
- board size 39 x 76 mm -> 249.8 x 170.3 mm

Commit message: Correccion final
Parts:
- removed the C1 at (231.6, 186.3)
- removed the C1 at (22.1, 186.9)
- removed the C1 at (229.9, 93.1)
- removed the C1 at (127.9, 187.4)
- removed the C1 at (177.0, 94.2)
- removed the C1 at (124.3, 93.9)
- removed the C1 at (75.2, 187.1)
- removed the C1 at (75.0, 94.3)
- removed the C1 at (178.9, 186.0)
- removed the C2 at (178.8, 172.6)
- removed the C2 at (229.8, 79.7)
- removed the C2 at (75.1, 173.7)
- removed the C2 at (127.8, 174.0)
- removed the C2 at (176.9, 80.8)
- removed the C2 at (231.5, 172.9)
- removed the C2 at (124.2, 80.5)
- removed the C2 at (22.0, 173.5)
- removed the C2 at (74.9, 80.9)
- removed the CAUDALIMETRO1 at (136.3, 27.1)
- removed the CAUDALIMETRO1 at (139.9, 120.6)
- removed the CAUDALIMETRO1 at (243.6, 119.5)
- removed the CAUDALIMETRO1 at (189.0, 27.4)
- removed the CAUDALIMETRO1 at (87.0, 27.5)
- removed the CAUDALIMETRO1 at (190.9, 119.2)
- removed the CAUDALIMETRO1 at (241.9, 26.3)
- removed the CAUDALIMETRO1 at (87.2, 120.3)
- removed the CAUDALIMETRO1 at (34.1, 120.1)
- removed the D1 at (199.6, 172.4)
- removed the D1 at (252.3, 172.7)
- removed the D1 at (197.7, 80.6)
- removed the D1 at (148.6, 173.8)
- removed the D1 at (42.8, 173.3)
- removed the D1 at (145.0, 80.3)
- removed the D1 at (95.7, 80.7)
- removed the D1 at (250.6, 79.5)
- removed the D1 at (95.9, 173.5)
- removed the H1 at (209.4, 184.4)
- removed the H1 at (105.5, 92.7)
- removed the H1 at (262.1, 184.7)
- removed the H1 at (158.4, 185.8)
- removed the H1 at (207.5, 92.6)
- removed the H1 at (105.7, 185.5)
- removed the H1 at (260.4, 91.5)
- removed the H1 at (154.8, 92.3)
- removed the H1 at (52.6, 185.3)
- removed the H2 at (74.9, 119.4)
- removed the H2 at (231.3, 118.6)
- removed the H2 at (74.7, 26.6)
- removed the H2 at (229.6, 25.4)
- removed the H2 at (21.8, 119.2)
- removed the H2 at (178.6, 118.3)
- removed the H2 at (127.6, 119.7)
- removed the H2 at (124.0, 26.2)
- removed the H2 at (176.7, 26.5)
- removed the J1 at (158.7, 180.3)
- removed the J1 at (207.8, 87.2)
- removed the J1 at (260.7, 86.0)
- removed the J1 at (209.7, 178.9)
- removed the J1 at (106.0, 180.1)
- removed the J1 at (155.1, 86.8)
- removed the J1 at (105.8, 87.2)
- removed the J1 at (52.9, 179.8)
- removed the J1 at (262.4, 179.2)
- removed the J2 at (30.8, 179.4)
- removed the J2 at (136.6, 179.9)
- removed the J2 at (133.0, 86.4)
- removed the J2 at (240.3, 178.8)
- removed the J2 at (83.9, 179.6)
- removed the J2 at (238.6, 85.6)
- removed the J2 at (185.7, 86.7)
- removed the J2 at (187.6, 178.5)
- removed the J2 at (83.7, 86.8)
- removed the J4 at (199.7, 183.2)
- removed the J4 at (148.7, 184.6)
- removed the J4 at (252.4, 183.5)
- removed the J4 at (95.8, 91.5)
- removed the J4 at (197.8, 91.4)
- removed the J4 at (250.7, 90.3)
- removed the J4 at (145.1, 91.1)
- removed the J4 at (96.0, 184.3)
- removed the J4 at (42.9, 184.1)
- removed the LCDOLED1 at (94.1, 117.9)
- removed the LCDOLED1 at (250.5, 117.1)
- removed the LCDOLED1 at (143.2, 24.7)
- removed the LCDOLED1 at (41.0, 117.7)
- removed the LCDOLED1 at (248.8, 23.9)
- removed the LCDOLED1 at (197.8, 116.8)
- removed the LCDOLED1 at (93.9, 25.1)
- removed the LCDOLED1 at (195.9, 25.0)
- removed the LCDOLED1 at (146.8, 118.2)
- removed the LDRMODULO1 at (195.8, 30.0)
- removed the LDRMODULO1 at (248.7, 28.9)
- removed the LDRMODULO1 at (197.7, 121.8)
- removed the LDRMODULO1 at (40.9, 122.7)
- removed the LDRMODULO1 at (93.8, 30.1)
- removed the LDRMODULO1 at (143.1, 29.7)
- removed the LDRMODULO1 at (94.0, 122.9)
- removed the LDRMODULO1 at (146.7, 123.2)
- removed the LDRMODULO1 at (250.4, 122.1)
- removed the Q1 at (248.6, 63.8)
- removed the Q1 at (146.6, 158.1)
- removed the Q1 at (93.7, 65.0)
- removed the Q1 at (40.8, 157.6)
- removed the Q1 at (143.0, 64.6)
- removed the Q1 at (197.6, 156.7)
- removed the Q1 at (93.9, 157.8)
- removed the Q1 at (195.7, 64.9)
- removed the Q1 at (250.3, 157.0)
- removed the R1 at (144.3, 70.4)
- removed the R1 at (249.9, 69.6)
- removed the R1 at (147.9, 163.9)
- removed the R1 at (251.6, 162.8)
- removed the R1 at (197.0, 70.7)
- removed the R1 at (95.2, 163.6)
- removed the R1 at (95.0, 70.8)
- removed the R1 at (42.1, 163.4)
- removed the R1 at (198.9, 162.5)
- removed the SENSORHUMEDAD1 at (136.5, 120.6)
- removed the SENSORHUMEDAD1 at (240.2, 119.5)
- removed the SENSORHUMEDAD1 at (187.5, 119.2)
- removed the SENSORHUMEDAD1 at (83.8, 120.3)
- removed the SENSORHUMEDAD1 at (30.7, 120.1)
- removed the SENSORHUMEDAD1 at (132.9, 27.1)
- removed the SENSORHUMEDAD1 at (185.6, 27.4)
- removed the SENSORHUMEDAD1 at (83.6, 27.5)
- removed the SENSORHUMEDAD1 at (238.5, 26.3)
- removed the U1 at (37.7, 150.6)
- removed the U1 at (90.6, 58.0)
- removed the U1 at (194.5, 149.7)
- removed the U1 at (192.6, 57.9)
- removed the U1 at (90.8, 150.8)
- removed the U1 at (245.5, 56.8)
- removed the U1 at (139.9, 57.6)
- removed the U1 at (143.5, 151.1)
- removed the U1 at (247.2, 150.0)
- removed the U2 at (22.1, 180.2)
- removed the U2 at (229.9, 86.4)
- removed the U2 at (75.0, 87.6)
- removed the U2 at (178.9, 179.3)
- removed the U2 at (75.2, 180.4)
- removed the U2 at (177.0, 87.5)
- removed the U2 at (127.9, 180.7)
- removed the U2 at (231.6, 179.6)
- removed the U2 at (124.3, 87.2)
- moved D1 105.3 mm to (143.6, 111.6)
- moved H1 105.3 mm to (153.4, 123.6)
- moved LCDOLED1 105.3 mm to (141.7, 56.0)
- moved LDRMODULO1 105.3 mm to (141.7, 61.0)
- moved R1 105.3 mm to (142.9, 101.7)
- moved SENSORHUMEDAD1 105.3 mm to (131.5, 58.3)
- moved U1 105.3 mm to (138.4, 88.9)
- moved C1 105.3 mm to (122.8, 125.2)
- moved C2 105.3 mm to (122.8, 111.8)
- moved CAUDALIMETRO1 105.3 mm to (134.9, 58.4)
- moved H2 105.3 mm to (122.6, 57.5)
- moved J1 105.3 mm to (153.7, 118.1)
- moved J2 105.3 mm to (131.6, 117.7)
- moved J4 105.3 mm to (143.7, 122.4)
- moved Q1 105.3 mm to (141.6, 95.9)
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Routing:
- net +5V: track 1406.2 -> 140.6 mm
- net /motor-: track 450.9 -> 45.1 mm
- net /A0: track 329.9 -> 33.0 mm
- net /SDA: track 325.2 -> 32.5 mm
- net /AUOT: track 289.6 -> 29.0 mm
- net /SERIAL: track 267.6 -> 26.8 mm
- net /SCL: track 238.1 -> 23.8 mm
- net +12V: track 147.9 -> 14.8 mm
- net +3.3V: track 145.2 -> 14.5 mm
- net Net-(Q1-B): track 32.7 -> 3.27 mm
- net /ON: track 32.0 -> 3.20 mm
Other:
- board size 249.8 x 170.3 mm -> 40.3 x 76 mm
